File: pcb/zilpzalp.kicad_sch (KiCad schematic)
At the start: 43 parts, among them SW1 SW_Push, SW10 SW_Push, SW11 SW_Push, SW12 SW_Push, SW13 SW_Push, SW14 SW_Push, SW15 SW_Push, SW16 SW_Push, SW17 SW_Push, SW18 SW_Push, SW19 SW_Push, SW2 SW_Push, SW20 SW_Push, SW21 SW_Push, SW22 SW_Push, SW23 SW_Push, SW24 SW_Push, SW25 SW_Push, SW26 SW_Push, SW27 SW_Push, SW28 SW_Push, SW3 SW_Push, SW4 SW_Push, SW5 SW_Push, SW6 SW_Push, SW7 SW_Push, SW8 SW_Push, SW9 SW_Push, U1 xiao

Commit message: change xiao footprint, silk slightly smaller
Parts:
- D01, D02, D03, D04, D05, D06, D07, D08, D09, D10, D11, D12, D13, D14: footprint Package_TO_SOT_SMD:SOT-23_Handsoldering -> BeiBob:SOT-23_Handsoldering
- SW1, SW10, SW11, SW12, SW13, SW14, SW15, SW16, SW17, SW18, SW19, SW2, SW20, SW21, SW22, SW23, SW24, SW25, SW26, SW27, SW28, SW3, SW4, SW5, SW6, SW7, SW8, SW9: footprint BeiBob:SW_Kailh_socket_PG1350_optional -> BeiBob:SW_Kailh_choc_hs_plus_solder_no_silk
- U1: footprint Kleeb MCU:xiao-ble-tht -> Kleeb MCU:xiao-tht
